File: creeLED.kicad_pcb (KiCad board)
At the start: 2 copper layers, 150 x 100 mm, 156 parts, among them J1 Conn_01x01, J10 Conn_01x01, J11 Conn_01x01, J12 Conn_01x01, J13 Conn_01x01, J14 Conn_01x01, J15 Conn_01x01, J16 Conn_01x01, J17 Conn_01x01, J18 Conn_01x01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

Commit message: v1.1
Parts:
- U1: value LM75B -> LM75A
Changed lines of the file:
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@@
   (net 131 "VD")
   (net 132 "GND")
-  (net 133 "Net-(U1-Pad1)")
-  (net 134 "Net-(U1-Pad2)")
-  (net 135 "Net-(U1-Pad3)")
+  (net 133 "Net-(J21-Pad1)")
+  (net 134 "Net-(J21-Pad2)")
+  (net 135 "Net-(J21-Pad3)")
   (footprint "Library:Cree_J-Series-2835-LED" (layer "F.Cu")
     (at 130 62)
@@
     )
     (pad "1" smd roundrect (at 0 -3) (size 5 2) (layers "F.Cu" "F.Paste" "F.Mask") (roundrect_rratio 0.25)
-      (net 133 "Net-(U1-Pad1)") (pinfunction "Pin_1") (pintype "passive"))
+      (net 133 "Net-(J21-Pad1)") (pinfunction "Pin_1") (pintype "passive"))
     (pad "2" smd roundrect (at 0 0) (size 5 2) (layers "F.Cu" "F.Paste" "F.Mask") (roundrect_rratio 0.25)
-      (net 134 "Net-(U1-Pad2)") (pinfunction "Pin_2") (pintype "passive"))
+      (net 134 "Net-(J21-Pad2)") (pinfunction "Pin_2") (pintype "passive"))
     (pad "3" smd roundrect (at 0 3) (size 5 2) (layers "F.Cu" "F.Paste" "F.Mask") (roundrect_rratio 0.25)
-      (net 135 "Net-(U1-Pad3)") (pinfunction "Pin_3") (pintype "passive"))
+      (net 135 "Net-(J21-Pad3)") (pinfunction "Pin_3") (pintype "passive"))
   )
   (footprint "Library:Cree_J-Series-2835-LED" (layer "F.Cu")
@@
       (net 131 "VD") (pintype "passive"))
     (pad "2" smd roundrect (at 0.9125 0) (size 0.975 0.95) (layers "F.Cu" "F.Paste" "F.Mask") (roundrect_rratio 0.25)
-      (net 135 "Net-(U1-Pad3)") (pintype "passive"))
+      (net 135 "Net-(J21-Pad3)") (pintype "passive"))
     (model "${KICAD6_3DMODEL_DIR}/Resistor_SMD.3dshapes/R_0603_1608Metric.wrl"
       (offset (xyz 0 0 0))
@@
       (effects (font (size 1 1) (thickness 0.15)))
     )
-    (fp_text value "LM75B" (at 0 3.4) (layer "F.Fab")
+    (fp_text value "LM75A" (at 0 3.4) (layer "F.Fab")
       (effects (font (size 1 1) (thickness 0.15)))
     )
@@
     (pad "" smd roundrect (at -0.6 0.775) (size 0.97 1.25) (layers "F.Paste") (roundrect_rratio 0.25))
     (pad "1" smd roundrect (at -2.65 -1.905) (size 1.6 0.6) (layers "F.Cu" "F.Paste" "F.Mask") (roundrect_rratio 0.25)
-      (net 133 "Net-(U1-Pad1)") (pinfunction "SDA") (pintype "bidirectional"))
+      (net 133 "Net-(J21-Pad1)") (pinfunction "SDA") (pintype "bidirectional"))
     (pad "2" smd roundrect (at -2.65 -0.635) (size 1.6 0.6) (layers "F.Cu" "F.Paste" "F.Mask") (roundrect_rratio 0.25)
-      (net 134 "Net-(U1-Pad2)") (pinfunction "SCL") (pintype "input"))
+      (net 134 "Net-(J21-Pad2)") (pinfunction "SCL") (pintype "input"))
     (pad "3" smd roundrect (at -2.65 0.635) (size 1.6 0.6) (layers "F.Cu" "F.Paste" "F.Mask") (roundrect_rratio 0.25)
-      (net 135 "Net-(U1-Pad3)") (pinfunction "O.S.") (pintype "open_collector"))
+      (net 135 "Net-(J21-Pad3)") (pinfunction "O.S.") (pintype "open_collector"))
     (pad "4" smd roundrect (at -2.65 1.905) (size 1.6 0.6) (layers "F.Cu" "F.Paste" "F.Mask") (roundrect_rratio 0.25)
       (net 132 "GND") (pinfunction "GND") (pintype "power_in"))
@@
       (net 131 "VD") (pintype "passive"))
     (pad "2" smd roundrect (at 0.9125 0) (size 0.975 0.95) (layers "F.Cu" "F.Paste" "F.Mask") (roundrect_rratio 0.25)
-      (net 134 "Net-(U1-Pad2)") (pintype "passive"))
+      (net 134 "Net-(J21-Pad2)") (pintype "passive"))
     (model "${KICAD6_3DMODEL_DIR}/Resistor_SMD.3dshapes/R_0603_1608Metric.wrl"
       (offset (xyz 0 0 0))
@@
       (net 131 "VD") (pintype "passive"))
     (pad "2" smd roundrect (at 0.9125 0) (size 0.975 0.95) (layers "F.Cu" "F.Paste" "F.Mask") (roundrect_rratio 0.25)
-      (net 133 "Net-(U1-Pad1)") (pintype "passive"))
+      (net 133 "Net-(J21-Pad1)") (pintype "passive"))
     (model "${KICAD6_3DMODEL_DIR}/Resistor_SMD.3dshapes/R_0603_1608Metric.wrl"
       (offset (xyz 0 0 0))
